File: PCB/CVTPCB.kicad_pcb (KiCad board)
At the start: 2 copper layers, 61 x 83.5 mm, 24 parts, among them J1 Infared, J2 TMP36, J3 Infared, J4 2x1, J5 TMP36, J7 SystemInput

Commit message: Add files via upload
Connections:
- U3 pad 19: /Ir2 -> /TMP36_1
- U3 pad 23: unconnected-(U3-D25-Pad23) -> /CanTX
- U3 pad 25: /CanTX -> unconnected-(U3-D27-Pad25)
- U3 pad 28: /TMP36_1 -> /Ir2
Routing:
- net /Ir2: track 24.5 -> 53.0 mm
- net /TMP36_1: track 45.4 -> 22.6 mm, vias 1 -> 0
- net /CanTX: track 37.7 -> 39.2 mm
- net /Ir1: track 25.9 -> 25.1 mm
- net /TMP36_2: track 28.9 -> 28.2 mm
- net (no net): track 0.00 -> 0.54 mm
- net /CanRX: track 35.7 -> 35.4 mm, vias 1 -> 0
Changed lines of the file:
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@@
 	(net 14 "unconnected-(U3-RX0-Pad12)")
 	(net 15 "unconnected-(U3-D5-Pad8)")
-	(net 16 "unconnected-(U3-D25-Pad23)")
+	(net 16 "unconnected-(U3-D27-Pad25)")
 	(net 17 "unconnected-(U3-EN-Pad16)")
 	(net 18 "unconnected-(U3-D32-Pad21)")
@@
 			(layers "*.Cu" "*.Mask")
 			(remove_unused_layers no)
-			(net 6 "/Ir2")
+			(net 8 "/TMP36_1")
 			(pinfunction "D34")
 			(pintype "bidirectional")
@@
 			(layers "*.Cu" "*.Mask")
 			(remove_unused_layers no)
-			(net 16 "unconnected-(U3-D25-Pad23)")
+			(net 24 "/CanTX")
 			(pinfunction "D25")
 			(pintype "bidirectional")
@@
 			(layers "*.Cu" "*.Mask")
 			(remove_unused_layers no)
-			(net 24 "/CanTX")
+			(net 16 "unconnected-(U3-D27-Pad25)")
 			(pinfunction "D27")
 			(pintype "bidirectional")
@@
 			(layers "*.Cu" "*.Mask")
 			(remove_unused_layers no)
-			(net 8 "/TMP36_1")
+			(net 6 "/Ir2")
 			(pinfunction "D13")
 			(pintype "bidirectional")
@@
 	)
 	(segment
+		(start 131 124)
+		(end 131 124.5)
+		(width 0.2)
+		(layer "F.Cu")
+		(net 0)
+	)
+	(segment
+		(start 131 124.5)
+		(end 130.96 124.5)
+		(width 0.2)
+		(layer "F.Cu")
+		(net 0)
+	)
+	(segment
 		(start 134.08 82)
 		(end 131 82)
@@
 	)
 	(segment
-		(start 141.54 117.5)
-		(end 141.54 110.54)
+		(start 143.336051 119.296051)
+		(end 141.54 117.5)
 		(width 0.2)
 		(layer "F.Cu")
@@
 	)
 	(segment
-		(start 141.54 110.54)
-		(end 138.5 107.5)
+		(start 142.04 117)
+		(end 141.54 117.5)
 		(width 0.2)
 		(layer "F.Cu")
@@
 	)
 	(segment
-		(start 138.5 107.5)
-		(end 134.53 107.5)
+		(start 147 117)
+		(end 142.04 117)
 		(width 0.2)
 		(layer "F.Cu")
@@
 	)
 	(segment
-		(start 141.54 117.5)
-		(end 146.5 117.5)
+		(start 131 115.5)
+		(end 131 86)
 		(width 0.2)
-		(layer "F.Cu")
+		(layer "B.Cu")
 		(net 6)
 	)
 	(segment
-		(start 144.703949 119.296051)
-		(end 147 117)
+		(start 133 117.5)
+		(end 131 115.5)
 		(width 0.2)
-		(layer "F.Cu")
+		(layer "B.Cu")
 		(net 6)
 	)
 	(segment
-		(start 134.53 107.5)
-		(end 134.255 107.225)
+		(start 131 86)
+		(end 132.5 84.5)
 		(width 0.2)
-		(layer "F.Cu")
+		(layer "B.Cu")
 		(net 6)
 	)
 	(segment
-		(start 146.5 117.5)
-		(end 147 117)
+		(start 134.12 84.5)
+		(end 134.255 84.365)
 		(width 0.2)
-		(layer "F.Cu")
+		(layer "B.Cu")
 		(net 6)
 	)
 	(segment
-		(start 144.08 66)
-		(end 146.5 66)
+		(start 132.5 84.5)
+		(end 134.12 84.5)
 		(width 0.2)
-		(layer "F.Cu")
-		(net 7)
+		(layer "B.Cu")
+		(net 6)
 	)
 	(segment
-		(start 137.5 84.57)
-		(end 135.165 86.905)
+		(start 141.54 117.5)
+		(end 133 117.5)
 		(width 0.2)
-		(layer "F.Cu")
-		(net 7)
+		(layer "B.Cu")
+		(net 6)
 	)
 	(segment
-		(start 142.5 66)
-		(end 137.5 71)
+		(start 144.08 66)
+		(end 146.5 66)
 		(width 0.2)
 		(layer "F.Cu")
@@
 	)
 	(segment
-		(start 144.08 66)
-		(end 142.5 66)
+		(start 139 83.5)
+		(end 135.595 86.905)
 		(width 0.2)
 		(layer "F.Cu")
@@
 	)
 	(segment
-		(start 137.5 71)
-		(end 137.5 84.57)
+		(start 139 71.08)
+		(end 139 83.5)
 		(width 0.2)
 		(layer "F.Cu")
@@
 	)
 	(segment
-		(start 135.165 86.905)
+		(start 135.595 86.905)
 		(end 134.255 86.905)
 		(width 0.2)
@@
 	)
 	(segment
-		(start 130.96 93.54)
-		(end 131 93.5)
+		(start 144.08 66)
+		(end 139 71.08)
 		(width 0.2)
 		(layer "F.Cu")
-		(net 8)
+		(net 7)
 	)
 	(segment
 		(start 130.96 125.5)
-		(end 130.96 93.54)
+		(end 131.5 124.96)
 		(width 0.2)
 		(layer "F.Cu")
@@
 	)
 	(segment
-		(start 128.04 125.5)
-		(end 130.96 125.5)
+		(start 131.5 124.96)
+		(end 131.5 109.98)
 		(width 0.2)
 		(layer "F.Cu")
 		(net 8)
 	)
-	(via
-		(at 131 93.5)
-		(size 0.6)
-		(drill 0.3)
-		(layers "F.Cu" "B.Cu")
-		(net 8)
-	)
 	(segment
-		(start 131 93.5)
-		(end 131 87.62)
+		(start 131.5 109.98)
+		(end 134.255 107.225)
 		(width 0.2)
-		(layer "B.Cu")
+		(layer "F.Cu")
 		(net 8)
 	)
 	(segment
-		(start 131 87.62)
-		(end 134.255 84.365)
+		(start 128.04 125.5)
+		(end 130.96 125.5)
 		(width 0.2)
-		(layer "B.Cu")
+		(layer "F.Cu")
 		(net 8)
 	)
@@
 	)
 	(segment
-		(start 143.606051 96.796051)
-		(end 145.402102 95)
+		(start 141.81 101.19)
+		(end 138.5 104.5)
 		(width 0.2)
 		(layer "F.Cu")
@@
 	)
 	(segment
-		(start 141.81 102.69)
-		(end 139.815 104.685)
+		(start 134.44 104.5)
+		(end 134.255 104.685)
 		(width 0.2)
 		(layer "F.Cu")
@@
 	)
 	(segment
-		(start 141.81 95)
-		(end 147.27 95)
+		(start 138.5 104.5)
+		(end 134.44 104.5)
+		(width 0.2)
+		(layer "F.Cu")
+		(net 9)
+	)
+	(segment
+		(start 143.606051 96.796051)
+		(end 145.402102 95)
 		(width 0.2)
 		(layer "F.Cu")
@@
 	(segment
 		(start 141.81 95)
-		(end 141.81 102.69)
+		(end 147.27 95)
 		(width 0.2)
 		(layer "F.Cu")
@@
 	)
 	(segment
-		(start 139.815 104.685)
-		(end 134.255 104.685)
+		(start 141.81 95)
+		(end 141.81 101.19)
 		(width 0.2)
 		(layer "F.Cu")
@@
 	)
 	(segment
-		(start 122.985 91.985)
-		(end 134.255 91.985)
+		(start 134.19 97)
+		(end 134.255 97.065)
 		(width 0.2)
 		(layer "F.Cu")
@@
 	)
 	(segment
-		(start 121.88 66)
-		(end 121.88 90.88)
+		(start 129 97)
+		(end 134.19 97)
 		(width 0.2)
 		(layer "F.Cu")
@@
 	)
 	(segment
-		(start 121.88 90.88)
-		(end 122.985 91.985)
+		(start 121.88 66)
+		(end 121.88 89.88)
 		(width 0.2)
 		(layer "F.Cu")
@@
 	)
 	(segment
-		(start 124.42 66)
-		(end 124.5 66.08)
+		(start 121.88 89.88)
+		(end 129 97)
 		(width 0.2)
 		(layer "F.Cu")
-		(net 25)
+		(net 24)
 	)
 	(segment
-		(start 124.5 66.08)
-		(end 124.5 90)
+		(start 124.42 89.42)
+		(end 129.525 94.525)
 		(width 0.2)
 		(layer "F.Cu")
 		(net 25)
 	)
-	(via
-		(at 124.5 90)
-		(size 0.6)
-		(drill 0.3)
-		(layers "F.Cu" "B.Cu")
-		(net 25)
-	)
 	(segment
-		(start 129.025 94.525)
-		(end 134.255 94.525)
+		(start 124.42 66)
+		(end 124.42 89.42)
 		(width 0.2)
-		(layer "B.Cu")
+		(layer "F.Cu")
 		(net 25)
 	)
 	(segment
-		(start 124.5 90)
-		(end 129.025 94.525)
+		(start 129.525 94.525)
+		(end 134.255 94.525)
 		(width 0.2)
-		(layer "B.Cu")
+		(layer "F.Cu")
 		(net 25)
 	)

Commit message: Add files via upload
Parts:
- removed R13: R, Resistor_THT:R_Axial_DIN0204_L3.6mm_D1.6mm_P5.08mm_Horizontal
- added R3: R, Resistor_THT:R_Axial_DIN0411_L9.9mm_D3.6mm_P12.70mm_Horizontal, F.Cu at (151.5, 96.0)
- J4: value 2x1 -> Conn_01x04_Pin; footprint Connector_PinHeader_1.00mm:PinHeader_1x02_P1.00mm_Vertical -> CVT:PowerBoard; moved to B.Cu
- J7: moved to F.Cu
- R1, R10, R11, R12, R2, R8, R9: footprint Resistor_THT:R_Axial_DIN0204_L3.6mm_D1.6mm_P5.08mm_Horizontal -> Resistor_THT:R_Axial_DIN0411_L9.9mm_D3.6mm_P12.70mm_Horizontal
- moved J7 39.1 mm to (156.5, 60.0), turned to 0 degrees
- moved R2 20.1 mm to (162.5, 113.8), turned to 90 degrees
- moved R11 16.5 mm to (124.5, 137.3), turned to 90 degrees
- moved R10 11.1 mm to (117.0, 124.7), turned to -90 degrees
- moved R12 10.7 mm to (162.5, 85.0), turned to -90 degrees
- moved RV2 10.4 mm to (149.8, 111.2), turned to 180 degrees
- moved J4 9.54 mm to (135.5, 105.2), turned to 90 degrees
- moved R8 9.00 mm to (155.5, 66.0), turned to -90 degrees
- moved R1 8.13 mm to (145.0, 121.0), turned to 0 degrees
- moved RV1 8.01 mm to (150.3, 101.2), turned to 180 degrees
- moved H1 6.73 mm to (154.0, 129.5)
- moved H4 1.58 mm to (106.0, 62.5)
- moved H2 1.50 mm to (107.5, 129.5)
- moved J2 1.50 mm to (130.5, 60.0)
- moved R9 0.50 mm to (139.5, 66.0)
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Connections:
- J1 pad 2: Net-(J1-IR-) -> /IrOut1
- J3 pad 2: Net-(J3-IR-) -> /IrOut2
- J7 pad 4: +12V -> /+12v
- R1 pad 1: Net-(J1-IR-) -> /IrOut1
- R1 pad 2: /Ir2 -> GND
- RV1 pad 1: /Ir1 -> GND
- RV1 pad 3: GND -> /IrOut2
- RV2 pad 1: /Ir2 -> GND
- RV2 pad 3: GND -> /IrOut1
- U3 pad 22: unconnected-(U3-D33-Pad22) -> /IrOut1
- U3 pad 26: unconnected-(U3-D14-Pad26) -> /IrOut2
Routing:
- net +5V: track 16.6 -> 144.8 mm, vias 4 -> 2
- net /+12v: track 0.00 -> 70.9 mm
- net /CanL: track 7.36 -> 58.2 mm
- net /IrOut1: track 0.00 -> 43.8 mm
- net /CanH: track 7.36 -> 51.2 mm
- net /IrOut2: track 0.00 -> 34.4 mm
- net Net-(J5-s): track 10.3 -> 26.3 mm
- net /Ir2: track 53.0 -> 37.9 mm, vias 0 -> 1
- net GND: track 17.1 -> 3.33 mm
- net /Ir1: track 25.1 -> 14.9 mm
- net /TMP36_2: track 28.2 -> 34.8 mm
- net /TMP36_1: track 22.6 -> 29.0 mm
- net Net-(J1-IR-): track 4.96 -> 0.00 mm
- net Net-(J3-IR-): track 4.69 -> 0.00 mm
- net Net-(J3-E+): track 4.46 -> 7.57 mm
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- removed copper zone on B.Cu, net +5V
Other:
- board size 61 x 83.5 mm -> 68 x 88 mm
- board text added: "12+"
- board text added: "CanH"
- board text added: "CanL"
- board text added: "RX"
- board text added: "TX"
- board text removed: "E-"
- board text removed: "Ir+"
